File: es32-kicad/workbench/workbench.kicad_pcb (KiCad board)
At the start: 4 copper layers, 99.9 x 99.7 mm, 67 parts, among them J1 GND|+5, J10 Rotary Encoder, J11 A[7..0], J2 [9..16], J3 B[0..7], J4 [17..24], J5 Conn_01x03_Socket, J6 Conn_01x03_Socket, J8 Conn_01x06_Socket, J9 [8..0]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

Commit message: adding pins for Leds. Silkscreen. logos. production files
Parts:
- removed J6: Conn_01x03_Socket, Connector_PinHeader_2.54mm:PinHeader_1x03_P2.54mm_Vertical
- added G***: LOGO, icons:che, F.Cu at (147.3, 125.2)
- added G***: LOGO, icons:depsi, B.Cu at (137.9, 73.9)
- added J7: Led-13-12-14, TerminalBlock_Phoenix:TerminalBlock_Phoenix_MKDS-3-3-5.08_1x03_P5.08mm_Horizontal, F.Cu at (100.5, 62.1)
- H3: footprint MountingHole:MountingHole_4.3mm_M4_Pad_Via -> MountingHole:MountingHole_4.3mm_M4_DIN965_Pad
- moved H3 16.5 mm to (119.5, 78.9)
- moved R35 15.9 mm to (114.7, 66.4), turned to 0 degrees
- moved J10 15.6 mm to (113.0, 51.6), turned to 180 degrees
- moved R22 13.2 mm to (114.7, 63.4), turned to 0 degrees
- moved R21 11.7 mm to (114.7, 60.3), turned to 0 degrees
- moved J1 5.25 mm to (100.2, 136.4), turned to -90 degrees
Connections:
- J1 pad 1: GND -> +5V
- J1 pad 2: +5V -> GND
- J10 pad 1: Net-(J10-Pin_1) -> GND
- J10 pad 4: GND -> Net-(J10-Pin_4)
- R21 pad 2: Net-(J10-Pin_3) -> Net-(J10-Pin_2)
- R22 pad 2: Net-(J10-Pin_2) -> Net-(J10-Pin_3)
- R35 pad 2: Net-(J10-Pin_1) -> Net-(J10-Pin_4)
- U11 pad 7: Net-(J10-Pin_3) -> Net-(J10-Pin_2)
- U11 pad 8: Net-(J10-Pin_2) -> Net-(J10-Pin_3)
- U11 pad 9: Net-(J10-Pin_1) -> Net-(J10-Pin_4)
Routing:
- net Net-(J10-Pin_1): track 38.4 -> 0.00 mm
- net Net-(J10-Pin_4): track 0.00 -> 35.1 mm
- net Net-(J7-Pin_1): track 4.16 -> 30.0 mm
- net Net-(J7-Pin_3): track 4.26 -> 29.3 mm
- net Net-(J7-Pin_2): track 4.16 -> 28.9 mm
- net Net-(J10-Pin_2): track 36.0 -> 21.6 mm
- net +5V: track 192.8 -> 200.7 mm
- net Net-(J10-Pin_3): track 28.4 -> 27.7 mm
Other:
- board text added: "https://github.com/crgarcia12/electronics-workbench-controller"
