File: PCB/workbench-01-jlcpcb/workbench.kicad_pcb (KiCad board)
At the start: 4 copper layers, 99.9 x 99.7 mm, 69 parts, among them J1 GND|+5, J10 Rotary Encoder, J11 A[7..0], J2 [9..16], J3 B[0..7], J4 [17..24], J5 Conn_01x03_Socket, J7 Led-13-12-14, J8 Conn_01x06_Socket, J9 [8..0]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

Commit message: V01 to JLC
Parts:
- C4: moved to B.Cu
- J1: value GND|+5 -> +5 | GND
- moved J1 85.9 mm to (186.1, 138.9), turned to 0 degrees
- moved C10 78.4 mm to (182.2, 134.5), turned to -90 degrees
- moved C9 71.8 mm to (178.9, 134.5), turned to -90 degrees
- moved C18 65.2 mm to (175.6, 134.5), turned to -90 degrees
- moved C13 58.6 mm to (172.3, 134.5), turned to -90 degrees
- moved C12 52.0 mm to (169.0, 134.5), turned to -90 degrees
- moved C11 45.4 mm to (165.7, 134.5), turned to -90 degrees
- moved C3 44.0 mm to (144.7, 129.8)
- moved J9 10.7 mm to (144.4, 138.9)
- moved J11 6.98 mm to (102.7, 138.9)
- moved C4 5.72 mm to (129.1, 91.9), turned to 0 degrees
- moved G*** 4.34 mm to (143.9, 122.6)
- moved C2 0.82 mm to (122.9, 96.5), turned to 0 degrees
Routing:
- net +5V: track 200.7 -> 167.5 mm
- net GND: track 44.9 -> 67.3 mm, vias 0 -> 3
- net Net-(J9-Pin_3): track 33.1 -> 45.6 mm
- net Net-(J9-Pin_2): track 39.6 -> 51.9 mm
- net Net-(J9-Pin_1): track 45.7 -> 57.6 mm
- net Net-(J9-Pin_4): track 27.5 -> 38.5 mm
- net Net-(J9-Pin_5): track 22.5 -> 31.0 mm
- net Net-(J9-Pin_8): track 22.4 -> 14.5 mm
- net Net-(J11-Pin_4): track 30.2 -> 24.4 mm
- net Net-(J11-Pin_5): track 37.8 -> 32.2 mm
- net Net-(J11-Pin_6): track 45.5 -> 39.9 mm
- net Net-(J11-Pin_7): track 53.1 -> 47.7 mm
- net Net-(J11-Pin_3): track 22.6 -> 17.2 mm
- net Net-(J11-Pin_8): track 60.7 -> 55.4 mm
- net Net-(J9-Pin_7): track 20.0 -> 16.5 mm
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Other:
- board text added: "locked"
