File: PCB/workbench-01-jlcpcb/workbench.kicad_sch (KiCad schematic)
At the start: 67 parts, among them J1 GND|+5, J10 Rotary Encoder, J11 A[7..0], J2 [9..16], J3 B[0..7], J4 [17..24], J5 Conn_01x03_Socket, J7 Led-13-12-14, J8 Conn_01x06_Socket, J9 [8..0]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

Commit message: V01 to JLC
Parts:
- J1: value GND|+5 -> +5 | GND
Changed lines of the file:
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@@
   (title_block
     (title "Workbench Controller")
-    (date "2023-05-26")
-    (rev "v1")
+    (date "2023-05-27")
+    (rev "V.20230527.01")
   )
   (junction (at 71.12 26.035) (diameter 0) (color 0 0 0 0)
@@
       (effects (font (size 1.27 1.27)) (justify left))
     )
-    (property "Value" "GND|+5" (at 64.77 10.16 90)
-      (effects (font (size 1.27 1.27)) (justify left) hide)
+    (property "Value" "+5 | GND" (at 60.96 13.97 90)
+      (effects (font (size 1.27 1.27)) (justify left))
     )
     (property "Footprint" "TerminalBlock_Phoenix:TerminalBlock_Phoenix_MKDS-3-2-5.08_1x02_P5.08mm_Horizontal" (at 54.61 16.51 0)
